File: dev_board/ml_dev_board.kicad_pcb (KiCad board)
At the start: 2 copper layers, 100 x 73.2 mm, 56 parts, among them J1 JTAG 3.3V, J2 Canon-Service-Connector, J3 USB_B_Mini, J4 Probe Connector, J5 canon_service_jumper_terminal, Q1 IRLML5203, U1 SN74AUP1T34DCK, U2 SN74AUP1T34DCK, U3 93LCxxBxxOT, U4 LD1117S33TR_SOT223, U5 FT4232H, U6 74HC595, Y1 12MHz

Commit message: dev board: rename JTAG 3.3V to JTAG 3v3
Parts:
- J1: value JTAG 3.3V -> JTAG 3v3
Changed lines of the file:
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@@
       (effects (font (size 1 1) (thickness 0.15)))
     )
-    (fp_text value "JTAG 3.3V" (at -0.02 -8.29 180) (layer F.SilkS)
+    (fp_text value "JTAG 3v3" (at -0.02 -8.29 180) (layer F.SilkS)
       (effects (font (size 1 1) (thickness 0.1875)))
     )
@@
   (segment (start 155.282 84.120466) (end 161.937456 77.46501) (width 0.25) (layer B.Cu) (net 1))
   (segment (start 155.282 84.582) (end 155.282 84.120466) (width 0.25) (layer B.Cu) (net 1))
-  (segment (start 109.148499 118.872) (end 107.1435 116.867001) (width 0.2) (layer F.Cu) (net 1))
+  (segment (start 109.148499 118.872) (end 107.1435 116.867001) (width 0.2) (layer F.Cu) (net 1) (status 20))
   (segment (start 118.747 118.872) (end 109.148499 118.872) (width 0.2) (layer F.Cu) (net 1))
   (via (at 118.11 97.536) (size 0.8) (drill 0.4) (layers F.Cu B.Cu) (net 2))
@@
   (segment (start 179.1 108) (end 179.1 105.25) (width 0.25) (layer F.Cu) (net 2) (status 30))
   (segment (start 173.9375 111.454) (end 173.9375 110.754) (width 0.2) (layer F.Cu) (net 2) (status 30))
-  (segment (start 170.0375 107.954) (end 170.0375 107.254) (width 0.2) (layer F.Cu) (net 2) (status 30))
+  (segment (start 170.0375 107.954) (end 170.0375 107.254) (width 0.2) (layer F.Cu) (net 2) (status 10))
   (via (at 176.6 114.25) (size 0.8) (drill 0.4) (layers F.Cu B.Cu) (net 2))
   (segment (start 176.55 114.3) (end 176.6 114.25) (width 0.25) (layer B.Cu) (net 2))
@@
   (segment (start 176.4775 102.63) (end 179.0175 102.63) (width 0.25) (layer F.Cu) (net 2) (status 30))
   (segment (start 170.32075 106.97075) (end 170.8655 106.426) (width 0.2) (layer F.Cu) (net 2))
-  (segment (start 170.0375 107.254) (end 170.32075 106.97075) (width 0.2) (layer F.Cu) (net 2) (status 10))
+  (segment (start 170.0375 107.254) (end 170.32075 106.97075) (width 0.2) (layer F.Cu) (net 2))
   (segment (start 168.942913 98.622913) (end 168.962913 98.622913) (width 0.25) (layer F.Cu) (net 2) (status 30))
   (segment (start 166.612913 100.952913) (end 168.942913 98.622913) (width 0.25) (layer F.Cu) (net 2) (status 30))
@@
   (segment (start 180.2 102.65) (end 180.85 102) (width 0.25) (layer F.Cu) (net 2))
   (segment (start 179.21 102.65) (end 180.2 102.65) (width 0.25) (layer F.Cu) (net 2) (status 10))
-  (segment (start 173.9375 107.954) (end 173.9375 107.254) (width 0.2) (layer F.Cu) (net 2) (status 30))
+  (segment (start 173.9375 107.954) (end 173.9375 107.254) (width 0.2) (layer F.Cu) (net 2) (status 10))
   (segment (start 173.9375 105.5875) (end 173.9375 107.954) (width 0.25) (layer F.Cu) (net 2) (status 20))
   (segment (start 170.0375 111.454) (end 170.0375 107.954) (width 0.2) (layer F.Cu) (net 2) (status 30))
@@
   (segment (start 185.8 76.7) (end 184.25 78.25) (width 0.2) (layer B.Cu) (net 3))
   (segment (start 184.25 78.95) (end 184.25 109.6) (width 0.25) (layer B.Cu) (net 3))
-  (segment (start 103.781001 116.867001) (end 106.17601 119.26201) (width 0.25) (layer F.Cu) (net 3))
+  (segment (start 103.781001 116.867001) (end 106.17601 119.26201) (width 0.25) (layer F.Cu) (net 3) (status 10))
   (segment (start 106.17601 119.26201) (end 108.57599 119.26201) (width 0.25) (layer F.Cu) (net 3))
   (segment (start 108.57599 119.26201) (end 118.550098 119.26201) (width 0.2) (layer F.Cu) (net 3))
@@
   (segment (start 163.95815 100.3) (end 166.229075 98.029075) (width 0.25) (layer B.Cu) (net 6))
   (segment (start 159.4 100.3) (end 163.95815 100.3) (width 0.25) (layer B.Cu) (net 6))
-  (segment (start 113.327001 114.046) (end 110.506 116.867001) (width 0.2) (layer F.Cu) (net 6))
+  (segment (start 113.327001 114.046) (end 110.506 116.867001) (width 0.2) (layer F.Cu) (net 6) (status 20))
   (segment (start 115.57 114.554) (end 116.078 114.046) (width 0.2) (layer F.Cu) (net 6))
-  (segment (start 115.57 115.9275) (end 115.57 114.554) (width 0.2) (layer F.Cu) (net 6))
+  (segment (start 115.57 115.9275) (end 115.57 114.554) (width 0.2) (layer F.Cu) (net 6) (status 10))
   (segment (start 116.078 114.046) (end 113.327001 114.046) (width 0.2) (layer F.Cu) (net 6))
   (segment (start 118.618 114.046) (end 116.078 114.046) (width 0.2) (layer F.Cu) (net 6))
@@
   (via (at 116.84 117.348) (size 0.8) (drill 0.4) (layers F.Cu B.Cu) (net 16))
   (segment (start 116.4355 117.7525) (end 116.84 117.348) (width 0.2) (layer F.Cu) (net 16))
-  (segment (start 115.57 117.7525) (end 116.4355 117.7525) (width 0.2) (layer F.Cu) (net 16))
+  (segment (start 115.57 117.7525) (end 116.4355 117.7525) (width 0.2) (layer F.Cu) (net 16) (status 10))
   (via (at 122.08 112.569) (size 0.8) (drill 0.4) (layers F.Cu B.Cu) (net 16))
   (segment (start 116.93299 117.25501) (end 116.84 117.348) (width 0.2) (layer B.Cu) (net 16))

Commit message: dev board: route unconnected ground pin
Routing:
- net GND: track 414.1 -> 417.7 mm
Changed lines of the file:
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@@
     (thickness 1.6)
     (drawings 102)
-    (tracks 1268)
+    (tracks 1270)
     (zones 0)
     (modules 56)
@@
   (segment (start 170.85 106.4105) (end 170.8655 106.426) (width 0.25) (layer B.Cu) (net 2))
   (segment (start 170.85 104.35) (end 170.85 106.4105) (width 0.25) (layer B.Cu) (net 2))
+  (segment (start 172.7 104.35) (end 173.9375 105.5875) (width 0.25) (layer F.Cu) (net 2))
+  (segment (start 170.85 104.35) (end 172.7 104.35) (width 0.25) (layer F.Cu) (net 2))
   (segment (start 183.1475 70.98) (end 184.56 72.3925) (width 0.25) (layer F.Cu) (net 3) (status 20))
   (segment (start 180.79 70.98) (end 183.1475 70.98) (width 0.25) (layer F.Cu) (net 3) (status 10))
@@
     (connect_pads (clearance 0.508))
     (min_thickness 0.254)
-    (fill (arc_segments 32) (thermal_gap 0.508) (thermal_bridge_width 0.508))
+    (fill yes (arc_segments 32) (thermal_gap 0.508) (thermal_bridge_width 0.508))
     (polygon
       (pts
@@
     (connect_pads (clearance 0.508))
     (min_thickness 0.254)
-    (fill (arc_segments 32) (thermal_gap 0.508) (thermal_bridge_width 0.508))
+    (fill yes (arc_segments 32) (thermal_gap 0.508) (thermal_bridge_width 0.508))
     (polygon
       (pts
