File: dev_board/ml_dev_board.kicad_pcb (KiCad board)
At the start: 2 copper layers, 100 x 73.2 mm, 56 parts, among them J1 JTAG 3v3, J2 Canon-Service-Connector, J3 USB_B_Mini, J4 Probe Connector, J5 canon_service_jumper_terminal, Q1 IRLML5203, U1 SN74AUP1T34DCK, U2 SN74AUP1T34DCK, U3 93LCxxBxxOT, U4 LD1117S33TR_SOT223, U5 FT4232H, U6 74HC595, Y1 12MHz

Commit message: dev board: added VCC ICU 1v8 + VCC MPU 3v3
Other:
- board text added: "VCC ICU 1.8V"
- board text added: "VCC MPU 3.3V"
Changed lines of the file:
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@@
-(kicad_pcb (version 20171130) (host pcbnew 5.1.8)
+(kicad_pcb (version 20171130) (host pcbnew 5.1.9)
   (general
     (thickness 1.6)
@@
     (34 B.Paste user)
     (35 F.Paste user)
-    (36 B.SilkS user hide)
+    (36 B.SilkS user)
     (37 F.SilkS user)
     (38 B.Mask user)
@@
     (effects (font (size 1.4 1.4) (thickness 0.2)))
   )
-  (gr_text NC (at 116.84 97.155 270) (layer F.SilkS)
+  (gr_text "VCC ICU 1.8V" (at 116.84 100.190714 -90) (layer F.SilkS)
     (effects (font (size 0.75 0.75) (thickness 0.1875)))
   )
-  (gr_text NC (at 134.62 97.155 270) (layer F.SilkS)
+  (gr_text "VCC MPU 3.3V" (at 134.62 100.440714 -90) (layer F.SilkS)
     (effects (font (size 0.75 0.75) (thickness 0.1875)))
   )
@@
     (connect_pads (clearance 0.508))
     (min_thickness 0.254)
-    (fill yes (arc_segments 32) (thermal_gap 0.508) (thermal_bridge_width 0.508))
+    (fill (arc_segments 32) (thermal_gap 0.508) (thermal_bridge_width 0.508))
     (polygon
       (pts
@@
     (connect_pads (clearance 0.508))
     (min_thickness 0.254)
-    (fill yes (arc_segments 32) (thermal_gap 0.508) (thermal_bridge_width 0.508))
+    (fill (arc_segments 32) (thermal_gap 0.508) (thermal_bridge_width 0.508))
     (polygon
       (pts

Commit message: dev board: pcb: 3.3V -> 3v3, 1.8V -> 1v8
Other:
- board text added: "RXDICU 1v8"
- board text added: "RXDMPU 3v3"
- board text added: "TXDICU 1v8"
- board text added: "TXDMPU 3v3"
- board text added: "VCC ICU 1v8"
- board text added: "VCC MPU 3v3"
- board text removed: "RXDICU 1.8V"
- board text removed: "RXDMPU 3.3V"
- board text removed: "TXDICU 1.8V"
- board text removed: "TXDMPU 3.3V"
- board text removed: "VCC ICU 1.8V"
- board text removed: "VCC MPU 3.3V"
Changed lines of the file:
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@@
     (effects (font (size 1.4 1.4) (thickness 0.2)))
   )
-  (gr_text "VCC ICU 1.8V" (at 116.84 100.190714 -90) (layer F.SilkS)
+  (gr_text "VCC ICU 1v8" (at 116.84 99.976428 -90) (layer F.SilkS)
     (effects (font (size 0.75 0.75) (thickness 0.1875)))
   )
-  (gr_text "VCC MPU 3.3V" (at 134.62 100.440714 -90) (layer F.SilkS)
+  (gr_text "VCC MPU 3v3" (at 134.62 100.226428 -90) (layer F.SilkS)
     (effects (font (size 0.75 0.75) (thickness 0.1875)))
   )
-  (gr_text "RXDMPU 3.3V" (at 132.08 100.190714 270) (layer F.SilkS)
+  (gr_text "RXDMPU 3v3" (at 132.08 99.976428 -90) (layer F.SilkS)
     (effects (font (size 0.75 0.75) (thickness 0.1875)))
   )
-  (gr_text "TXDMPU 3.3V" (at 129.54 100.101428 270) (layer F.SilkS)
+  (gr_text "TXDMPU 3v3" (at 129.54 99.887143 -90) (layer F.SilkS)
     (effects (font (size 0.75 0.75) (thickness 0.1875)))
   )
@@
     (effects (font (size 0.75 0.75) (thickness 0.1875)))
   )
-  (gr_text "TXDICU 1.8V" (at 121.92 99.851428 270) (layer F.SilkS)
+  (gr_text "TXDICU 1v8" (at 121.92 99.637143 -90) (layer F.SilkS)
     (effects (font (size 0.75 0.75) (thickness 0.1875)))
   )
-  (gr_text "RXDICU 1.8V" (at 119.38 99.940714 270) (layer F.SilkS)
+  (gr_text "RXDICU 1v8" (at 119.38 99.726428 -90) (layer F.SilkS)
     (effects (font (size 0.75 0.75) (thickness 0.1875)))
   )

Commit message: dev board: pcb: update version number to v2.0
Other:
- board text added: "Magic Lantern Dev Kit v2.00 - 03/2021"
- board text removed: "Magic Lantern Dev Kit v1.00 - 10/2020"
Changed lines of the file:
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@@
     )
   )
-  (gr_text "Magic Lantern Dev Kit\nv1.00 - 10/2020" (at 133.2 117.95) (layer F.SilkS)
+  (gr_text "Magic Lantern Dev Kit\nv2.00 - 03/2021" (at 133.2 117.95) (layer F.SilkS)
     (effects (font (size 1 1) (thickness 0.15)))
   )

Commit message: update kicad version
Connections:
- J5 pad 11: (no net) -> /VCC_ICU_1v8
- J5 pad 15: (no net) -> unconnected-(J5-Pin_15-Pad15)
- J5 pad 18: (no net) -> /VCC_MPU_3v3
- U5 pad 21: (no net) -> unconnected-(U5-ADBUS4-Pad21)
- U5 pad 22: (no net) -> unconnected-(U5-ADBUS5-Pad22)
- U5 pad 23: (no net) -> unconnected-(U5-ADBUS6-Pad23)
- U5 pad 24: (no net) -> unconnected-(U5-ADBUS7-Pad24)
- U5 pad 26: (no net) -> /FTDI/RXFPU
- U5 pad 27: (no net) -> /FTDI/TXFPU
- U5 pad 28: (no net) -> unconnected-(U5-BDBUS2-Pad28)
- U5 pad 29: (no net) -> unconnected-(U5-BDBUS3-Pad29)
- U5 pad 30: (no net) -> unconnected-(U5-BDBUS4-Pad30)
- U5 pad 32: (no net) -> unconnected-(U5-BDBUS5-Pad32)
- U5 pad 33: (no net) -> unconnected-(U5-BDBUS6-Pad33)
- U5 pad 34: (no net) -> unconnected-(U5-BDBUS7-Pad34)
- U5 pad 36: (no net) -> unconnected-(U5-~{SUSPEND}-Pad36)
- U5 pad 40: (no net) -> unconnected-(U5-CDBUS2-Pad40)
- U5 pad 41: (no net) -> unconnected-(U5-CDBUS3-Pad41)
- U5 pad 43: (no net) -> unconnected-(U5-CDBUS4-Pad43)
- U5 pad 44: (no net) -> unconnected-(U5-CDBUS5-Pad44)
- U5 pad 45: (no net) -> unconnected-(U5-CDBUS6-Pad45)
- U5 pad 46: (no net) -> unconnected-(U5-CDBUS7-Pad46)
- U5 pad 53: (no net) -> unconnected-(U5-DDBUS2-Pad53)
- U5 pad 54: (no net) -> unconnected-(U5-DDBUS3-Pad54)
- U5 pad 55: (no net) -> unconnected-(U5-DDBUS4-Pad55)
- U5 pad 57: (no net) -> unconnected-(U5-DDBUS5-Pad57)
- U5 pad 58: (no net) -> unconnected-(U5-DDBUS6-Pad58)
- U5 pad 59: (no net) -> unconnected-(U5-DDBUS7-Pad59)
- U6 pad 1: (no net) -> unconnected-(U6-QB-Pad1)
- U6 pad 15: (no net) -> unconnected-(U6-QA-Pad15)
- U6 pad 2: (no net) -> unconnected-(U6-QC-Pad2)
- U6 pad 3: (no net) -> unconnected-(U6-QD-Pad3)
- U6 pad 9: (no net) -> unconnected-(U6-QH'-Pad9)
Other:
- net class Default removed
